File: H17R10/H17R10.brd (EAGLE design)
At the start: 60.6 x 60 mm, 64 parts, among them P1 HEXABIT__X3_NO_P1_P2_P3_P4, U1 STM32F091RBT6STMICROELECTRONI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, U2 POWERSTEP01, U5 TEXAS_INSTRUMENTS_ISO7741DBQR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, U6 TEXAS_INSTRUMENTS_ISO7742DBQR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, X1 XTALL_CSTCE8M00G52

Commit message: R24  added
Parts:
- removed C800: 100nF, Hexabitz:C-0603
- added C16, C17, C18, C19: 100nF, HEXABITZ_RCLS:C-0603
- added C50: 100nF, Hexabitz:C-0603
- added J1, SPI_MTR: 3-644456-2, HEXABITZ_USER_INTERFACE_PARTS:TE_3-644456-2
- added R20: 330, HEXABITZ_RCLS:R-0603
- added R22, R24, R27, R28: DNP, HEXABITZ_RCLS:R-0805
- added R23, R8: 0R, HEXABITZ_RCLS:R-0603
- added R5, R6, R7: DNP, HEXABITZ_RCLS:R-0603
- C5: value NP -> DNP; device HEXABITZ_RCLS:C-0603 -> HEXABITZ_RCLS:C-0805
- R3: value 330 -> 0R
- R4: value 0R -> DNP
- moved U5 151.9 mm to (24.8, -20.0)
- moved U6 129.1 mm to (24.4, -37.1)
- moved R4 98.4 mm to (-37.8, -181.9)
- moved R3 97.1 mm to (-37.8, -172.4)
- moved C5 74.9 mm to (-44.8, -201.9)
- moved R 60.0 mm to (21.3, -30.1)
- moved R100 14.2 mm to (-7.04, -20.9)
- moved D0 14.2 mm to (-9.42, -20.5)
- moved U1 2.86 mm to (11.4, -28.3)
- moved X1 1.59 mm to (20.6, -26.7)
- renumbered R99 to R50
Connections:
- removed net N$24: U5.13
- removed net N$25: U5.12
- removed net N$26: U5.11
- removed net N$27: U6.4
- removed net N$28: U6.5
- removed net N$29: U6.6
- removed net N$30: U6.12
- removed net N$31: U6.11
- removed net N$32: U6.14
- removed net N$33: U6.13
- new net MC_BUSY/SYNC: U1.22, U6.3
- new net MC_CK: U1.55, U5.4
- new net MC_CS: U1.58, U5.3
- new net MC_FLAG: U1.23, U6.4
- new net MC_MISO: U1.56, U5.6
- new net MC_MOSI: U1.57, U5.5
- new net MC_STBY/RESET: U1.25, U6.6
- new net MS_STCK: U1.24, U6.5
- new net SW: J1.1, U2.18
- net ADC_IN: now also R27.2, R28.1
- net BUSY/SYNC: now also U6.12
- net CK: now also U5.13
- net CS: now also U5.14
- net FLAG: now also U6.11
- net GND: now also C17.2, C19.2, C50.2; no longer C800.2
- net GND1: now also C16.2, C18.2, J1.2, R27.1, X2.2
- net N$1: now also R20.2; no longer R3.2
- net N$14: now also R20.1; no longer R3.1
- net N$18: now also R3.1, U5.12; no longer U6.3
- net N$19: now also R8.1, U5.11; no longer U5.3
- net N$20: now also R4.1, R6.1, SPI_MTR.2; no longer U5.4
- net N$21: now also R5.1, R7.1, SPI_MTR.1; no longer U5.5
- net N$22: now also R22.2, U2.64; no longer U5.6
- net N$23: now also R22.1, U2.63; no longer U5.14
- net N$8: now also R24.1
- net OUTA1: now also X3.1
- net OUTA2: now also X3.2
- net OUTB1: now also X4.1
- net OUTB2: now also X4.2
- net R1: now also C50.1; no longer C800.1
- net SDI: now also R3.2, R4.2, R5.2
- net SDO: now also R6.2, R7.2, R8.2
- net STBY/RESET: now also U6.13
- net STCK: now also U6.14
- net UART5_RX: no longer U1.56
- net UART5_TX: no longer U1.55
- net VDD: now also C16.1, C17.1, C18.1, C19.1
- net VSREG: now also R23.2, R24.2; no longer R4.2
- net VSS: now also R23.1, R28.2, X2.1; no longer R4.1
Routing:
- net N$6: track 2.68 -> 3.95 mm
- net N$5: track 2.68 -> 3.95 mm
- added copper zone on layer 1, net VDD

Commit message: finished board >>> unchecked
Parts:
- removed C100: 10nF, Hexabitz:C-0603
- removed C200: 1.00uF, Hexabitz:C-0805-POL
- removed C300, C50, C500, C600, C900: 100nF, Hexabitz:C-0603
- removed C400, C700: 4.7uF, Hexabitz:C-0805-POL
- removed J1: 3-644456-2, HEXABITZ_USER_INTERFACE_PARTS:TE_3-644456-2
- removed R100: 270.0R, Hexabitz:R-0603
- removed R50: 10.0K, Hexabitz:R-0603
- removed U5: TEXAS_INSTRUMENTS_ISO7741DBQRTEXAS_INSTRUMENTS_ISO7741DBQR_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, Texas Instruments - ISO7741DBQR:TEXAS_INSTRUMENTS_ISO7741DBQR_3
- added C21: 100nF, HEXABITZ_RCLS:C-0603
- added C22: 1.00uF, Hexabitz:C-0805-POL
- added C23, C24: 4.7uF, Hexabitz:C-0805-POL
- added C25: 10nF, Hexabitz:C-0603
- added C26, C27, C28, C29: 100nF, Hexabitz:C-0603
- added D11: RED, HEXABITZ_USER_INTERFACE_PARTS:VLMS1300-GS08
- added D12, D13: Green, HEXABITZ_USER_INTERFACE_PARTS:VLMTG1300-GS08
- added EMG_SW: 3-644456-2, HEXABITZ_USER_INTERFACE_PARTS:TE_3-644456-2
- added R10, R11, R31, R9: 270.0R, HEXABITZ_RCLS:R-0603
- added R32: 10.0K, Hexabitz:R-0603
- added R33, R34: DNP, HEXABITZ_RCLS:R-0603
- added U3: TEXAS_INSTRUMENTS_ISO7741DBQRTEXAS_INSTRUMENTS_ISO7741DBQR_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, HEXABITZ_ICs:TEXAS_INSTRUMENTS_ISO7741DBQR_0
- C5: device HEXABITZ_RCLS:C-0805 -> HEXABITZ_RCLS:C-0603
- D0: value VLMS1300-GS08 -> RED; device Hexabitz:VLMS1300-GS08 -> HEXABITZ_USER_INTERFACE_PARTS:VLMS1300-GS08
- D2: value red -> RED; device HEXABITZ_USER_INTERFACE_PARTS:CHIP-LED0805 -> HEXABITZ_USER_INTERFACE_PARTS:VLMS1300-GS08
- D3, D4, D5, D6, D7: value yallow -> YELLOW; device HEXABITZ_USER_INTERFACE_PARTS:CHIP-LED0805 -> HEXABITZ_USER_INTERFACE_PARTS:VLMY1300-GS08
- D8: value green -> Green; device HEXABITZ_USER_INTERFACE_PARTS:CHIP-LED0805 -> HEXABITZ_USER_INTERFACE_PARTS:VLMTG1300-GS08
- P1: value HEXABIT__X3_NO_P1_P2_P3_P4 -> HEXABIT__X3_NO_P1_P2_P3_P4_P5_P6_P11_P12; device hexabitz_connectors:HEXABIT_17.32_X3_NO_P1_P2_P3_P4 -> hexabitz_connectors:HEXABIT_17.32_X3_NO_P1_P2_P3_P4_P5_P6_P11_P12
- R22, R27: device HEXABITZ_RCLS:R-0805 -> HEXABITZ_RCLS:R-0603
- U2: value POWERSTEP01 -> (none)
- moved R24 250.4 mm to (-8.33, 6.11), turned to 270 degrees
- moved R22 229.9 mm to (-11.6, 8.73), turned to 270 degrees
- moved R7 220.5 mm to (-15.0, 23.1), flipped to the bottom, turned to 210 degrees
- moved R6 218.5 mm to (-13.5, 25.7), flipped to the bottom, turned to 210 degrees
- moved SPI_MTR 210.8 mm to (-24.1, 15.2), turned to 60 degrees
- moved R5 209.8 mm to (-19.8, 22.4), flipped to the bottom, turned to 30 degrees
- moved R4 207.8 mm to (-18.3, 25.0), flipped to the bottom, turned to 30 degrees
- moved R27 201.6 mm to (-9.37, -13.9), turned to 180 degrees
- moved R3 201.1 mm to (-16.8, 27.6), flipped to the bottom, turned to 30 degrees
- moved R8 198.8 mm to (-16.5, 20.5), flipped to the bottom, turned to 210 degrees
- moved R28 196.3 mm to (-13.0, -14.5), turned to 180 degrees
- moved C5 192.1 mm to (-13.1, -12.5), turned to 180 degrees
- moved C19 176.6 mm to (-36.7, 8.81), turned to 180 degrees
- moved C18 165.4 mm to (-27.9, 2.54)
- moved C16 162.1 mm to (-26.2, 8.65)
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Connections:
- removed net SPI2_CS: U1.33
- removed net UART5_RX: P1.PAD_PD9
- removed net UART5_TX: P1.PAD_PU9
- removed net VDDIO: U2.13
- new net FORWARD: R10.2, U1.33
- new net N$24: D12.A, R10.1
- new net N$25: D13.A, R11.1
- new net REVERSED: R11.2, U1.45
- new net STOPPED: R9.2, U1.44
- net B1: now also R32.2; no longer R50.2
- net BUSY/SYNC: now also U6.14; no longer U6.12
- net CK: now also U3.13; no longer U5.13
- net CS: now also U3.14; no longer U5.14
- net FLAG: now also U6.13; no longer U6.11
- net GND: now also C21.2, C22.2, C23.2, C24.2, C25.2, C26.2, C27.2, C28.2, C29.2, D11.C, D12.C, D13.C, R32.1, U1.53, U1.54, U3.2, U3.8; no longer C100.2, C200.2, C300.2, C400.2, C50.2, C500.2, C600.2, C700.2, C900.2, P1.PAD_PD13, P1.PAD_PD14, P1.PAD_PD15, P1.PAD_PD16, P1.PAD_PD18, P1.PAD_PD5, R50.1, U1.44, U1.45, U5.2, U5.8
- net GND1: now also EMG_SW.2, U3.15, U3.9; no longer J1.2, U5.15, U5.9
- net MC_BUSY/SYNC: now also U1.25; no longer U1.22
- net MC_CK: now also U3.4; no longer U5.4
- net MC_CS: now also U3.3; no longer U5.3
- net MC_FLAG: now also U1.24; no longer U1.23
- net MC_MISO: now also R33.1, U3.6; no longer U5.6
- net MC_MOSI: now also R34.1, U3.5; no longer U5.5
- net MC_STBY/RESET: now also U1.22; no longer U1.25
- net MS_STCK: now also U1.23; no longer U1.24
- net N$11: now also D11.A, R9.1; no longer R16.2, R17.2, R18.2, R19.2
- net N$18: now also U3.12; no longer U5.12
- net N$19: now also U3.11; no longer U5.11
- net N$3: now also R31.2; no longer R100.2
- net N$4: now also R31.1; no longer R100.1
- net OUTA1: now also R16.2, X3.2; no longer X3.1
- net OUTA2: now also R17.2, X3.1; no longer X3.2
- net OUTB1: now also R18.2
- net OUTB2: now also R19.2
- net R1: now also C21.1; no longer C50.1
- net STBY/RESET: now also U6.11; no longer U6.13
- net STCK: now also U6.12; no longer U6.14
- net SW: now also EMG_SW.1; no longer J1.1
- net UART1_RX*: now also P1.PAD_PD2; no longer P1.PAD_PD8
- net UART1_TX*: now also P1.PAD_PU2; no longer P1.PAD_PU8
- net UART3_RX: no longer P1.PAD_PD2
- net UART3_TX: no longer P1.PAD_PU2
- net UART4_RX: now also P1.PAD_PD8, U1.52; no longer P1.PAD_PD6, U1.15
- net UART4_TX: now also P1.PAD_PU8, U1.51; no longer P1.PAD_PU6, U1.14
- net UART7_RX: no longer P1.PAD_PD7
- net UART7_TX: no longer P1.PAD_PU7
- net UART8_RX: no longer P1.PAD_PD4
- net UART8_TX: no longer P1.PAD_PU4
- net VCCIO: now also C1.1, C16.1, C18.1, C4.1, R13.2, R14.2, R15.1, R21.2, R25.2, R26.2, U2.13, U3.10, U3.16; no longer U5.10, U5.16
- net VDD: now also C22.1, C23.1, C24.1, C25.1, C26.1, C27.1, C28.1, C29.1, R33.2, R34.2, U3.1, U3.7; no longer C1.1, C100.1, C16.1, C18.1, C200.1, C300.1, C4.1, C400.1, C500.1, C600.1, C700.1, C900.1, P1.PAD_PU13, P1.PAD_PU14, P1.PAD_PU15, P1.PAD_PU16, P1.PAD_PU18, P1.PAD_PU5, R13.2, R14.2, R15.1, R21.2, R25.2, R26.2, U5.1, U5.7
Routing:
- net VSS: track 0.00 -> 95.1 mm, vias 0 -> 20
- net VCCIO: track 0.00 -> 57.5 mm, vias 0 -> 1
- net SDO: track 0.00 -> 37.1 mm, vias 0 -> 2
- net SDI: track 0.00 -> 34.9 mm, vias 0 -> 2
- net GND: track 0.00 -> 33.7 mm, vias 0 -> 5
- net N$18: track 0.00 -> 29.6 mm, vias 0 -> 2
- net GND1: track 0.00 -> 29.2 mm, vias 0 -> 67
- net REVERSED: track 0.00 -> 25.9 mm, vias 0 -> 2
- net OUTB1: track 0.00 -> 25.7 mm, vias 0 -> 4
- net BUSY/SYNC: track 0.00 -> 24.9 mm, vias 0 -> 2
- net STOPPED: track 0.00 -> 24.4 mm, vias 0 -> 2
- net SENSE_A: track 0.00 -> 23.9 mm
- net N$1: track 0.00 -> 23.6 mm
- net FORWARD: track 0.00 -> 23.5 mm, vias 0 -> 2
- net OUTA1: track 0.00 -> 23.0 mm, vias 0 -> 4
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- added copper zone on layer 1, net GND1
- added copper zone on layer 16, net GND1
- added copper zone on layer 2, net GND1
- added copper zone on layer 16, net OUTA1
- added copper zone on layer 16, net OUTA2
- added copper zone on layer 16, net OUTB1
- added copper zone on layer 16, net OUTB2
- added copper zone on layer 16, net VSS
- added copper zone on layer 3, net VSS
- removed copper zone on layer 1, net AGND
- removed copper zone on layer 2, net AGND
- removed copper zone on layer 15, net GND
Other:
- board text added: "+"
- board text added: "-"
- board text added: "A1"
- board text added: "A2"
- board text added: "B1"
- board text added: "B2"
- board text added: "H17R10"
- board text added: "P10"
- board text added: "P9"
- board text added: "P9*"
- board text added: "isolation"
- board text removed: "H26R10"
- board text removed: "P1"
- board text removed: "P2*"
- board text removed: "P3"
- board text removed: "P4"
- board text removed: "P5"
- board text removed: "P6*"

Commit message: no message
Parts:
- added P3, P4, P5, P6, VCCIO, VCCIO1, VS: PAD4, HEXABITZ_CONNECTION_PARTS:PAD4
- moved R10 1.12 mm to (-42.5, -6.51), turned to 270 degrees
- moved C1 0.79 mm to (-28.7, 12.0)
- renumbered D11 to S, D12 to CCW, D13 to CW, D2 to FLT, D3 to A1, D4 to A2, D5 to B1, D6 to B2, D7 to BZY, D8 to PWR, U6 to U4
Connections:
- removed net SPI2_MISO: U1.35
- removed net SPI2_SCK: U1.34
- net GND: now also P5.P$1
- net GND1: now also P6.P$1
- net VCCIO: now also VCCIO.P$1, VCCIO1.P$1
- net VDD: now also P4.P$1
- net VSS: now also VS.P$1
Routing:
- net VSS: track 95.1 -> 99.6 mm
- net VCCIO: track 57.5 -> 59.8 mm
- net N$24: track 3.17 -> 4.55 mm
- net FORWARD: track 23.5 -> 22.3 mm
- net GND1: track 29.2 -> 30.1 mm, vias 67 -> 66
