File: H17R10/H17R10.sch (EAGLE design)
At the start: 64 parts, among them P1 HEXABIT__X3_NO_P1_P2_P3_P4, U1 STM32F091RBT6STMICROELECTRONI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, U2 POWERSTEP01, U5 TEXAS_INSTRUMENTS_ISO7741DBQR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, U6 TEXAS_INSTRUMENTS_ISO7742DBQR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, X1 XTALL_CSTCE8M00G52

Commit message: R24  added
Parts:
- added C16, C17, C18, C19: 100nF, HEXABITZ_RCLS:C-0603
- added J1, SPI_MTR: 3-644456-2, HEXABITZ_USER_INTERFACE_PARTS:3-644456-2
- added R20: 330, HEXABITZ_RCLS:R-0603
- added R22, R24, R27, R28: DNP, HEXABITZ_RCLS:R-0805
- added R23, R8: 0R, HEXABITZ_RCLS:R-0603
- added R5, R6, R7: DNP, HEXABITZ_RCLS:R-0603
- C5: value NP -> DNP; device HEXABITZ_RCLS:C-0603 -> HEXABITZ_RCLS:C-0805; CAPACITANCE NP -> (none); MFN NP -> (none); MPN NP(0603) -> (none)
- R3: value 330 -> 0R; DESCRIPTION (none) -> RC Series 0603 0.1 W 0 Ohm Jumper Surface Mount Thick Film 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; MPN RC0603JR-07330RL -> RC0603JR-070RL; OCTOPART_URL https://octopart.com/rc0603jr-07330rl-yageo-39803615?r=sp -> https://octopart.com/rc0603jr-070rl-yageo-1241539?r=sp; RESISTANCE 330 -> (none)
- R4: value 0R -> DNP; MFN Yageo -> (none); MPN RC0603JR-070RL -> DNP; OCTOPART_URL https://octopart.com/rc0603jr-070rl-yageo-1241539?r=sp -> (none)
- renumbered C800 to C50, R99 to R50
Connections:
- removed net N$24: U5.OUTB
- removed net N$25: U5.OUTC
- removed net N$26: U5.IND
- removed net N$27: U6.INB
- removed net N$28: U6.OUTC
- removed net N$29: U6.OUTD
- removed net N$30: U6.INC
- removed net N$31: U6.IND
- removed net N$32: U6.OUTA
- removed net N$33: U6.OUTB
- new net MC_BUSY/SYNC: U1.PA6, U6.INA
- new net MC_CK: U1.PB3, U5.INB
- new net MC_CS: U1.PB6, U5.INA
- new net MC_FLAG: U1.PA7, U6.INB
- new net MC_MISO: U1.PB4, U5.OUTD
- new net MC_MOSI: U1.PB5, U5.INC
- new net MC_STBY/RESET: U1.PC5, U6.OUTD
- new net MS_STCK: U1.PC4, U6.OUTC
- new net SW: J1.1, U2A.SW
- net ADC_IN: now also R27.2, R28.1
- net BUSY/SYNC: now also U6.INC
- net CK: now also U5.OUTB
- net CS: now also U5.OUTA
- net FLAG: now also U6.IND
- net GND: now also C17.2, C19.2
- net GND1: now also C16.2, C18.2, J1.2, R27.1, X2-2.KL
- net N$1: now also R20.2; no longer R3.2
- net N$14: now also R20.1; no longer R3.1
- net N$18: now also R3.1, U5.OUTC; no longer U6.INA
- net N$19: now also R8.1, U5.IND; no longer U5.INA
- net N$20: now also R4.1, R6.1, SPI_MTR.2; no longer U5.INB
- net N$21: now also R5.1, R7.1, SPI_MTR.1; no longer U5.INC
- net N$22: now also R22.2, U2B.OSCOUT; no longer U5.OUTD
- net N$23: now also R22.1, U2B.OSCIN; no longer U5.OUTA
- net N$8: now also R24.1
- net OUTA1: now also X3-1.KL
- net OUTA2: now also X3-2.KL
- net OUTB1: now also X4-1.KL
- net OUTB2: now also X4-2.KL
- net SDI: now also R3.2, R4.2, R5.2
- net SDO: now also R6.2, R7.2, R8.2
- net STBY/RESET: now also U6.OUTB
- net STCK: now also U6.OUTA
- net UART5_RX: no longer U1.PB4
- net UART5_TX: no longer U1.PB3
- net VDD: now also C16.1, C17.1, C18.1, C19.1
- net VSREG: now also R23.2, R24.2; no longer R4.2
- net VSS: now also R23.1, R28.2, X2-1.KL; no longer R4.1
Other:
- note added: "BOOT STRAP"
- note added: "Control pins"
- note added: "GND is isolated"
- note added: "POWER WITH 80v MAX PULL 10A RMS MAX"
- note added: "SPI"
- note added: "Vccio = 3.3v (output)"
- note added: "Vs=80v max"
- note added: "high_power"
- note added: "logic"
- note removed: "GND_IS_DEFRRENT"
- moved on the sheet: C1, C10, C11, C12, C13, C14, C15, C2, C3, C4, C6, C7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

Commit message: finished board >>> unchecked
Parts:
- removed C100: 10nF, Hexabitz:C-0603
- removed C200: 1.00uF, Hexabitz:C-0805-POL
- removed C300, C50, C500, C600, C900: 100nF, Hexabitz:C-0603
- removed C400, C700: 4.7uF, Hexabitz:C-0805-POL
- removed R100: 270.0R, Hexabitz:R-0603
- removed U5: TEXAS_INSTRUMENTS_ISO7741DBQRTEXAS_INSTRUMENTS_ISO7741DBQR_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, Texas Instruments - ISO7741DBQR:TEXAS_INSTRUMENTS_ISO7741DBQRTEXAS_INSTRUMENTS_ISO7741DBQR_0_3
- added C21: 100nF, HEXABITZ_RCLS:C-0603
- added C22: 1.00uF, Hexabitz:C-0805-POL
- added C23, C24: 4.7uF, Hexabitz:C-0805-POL
- added C25: 10nF, Hexabitz:C-0603
- added C26, C27, C28, C29: 100nF, Hexabitz:C-0603
- added D11: RED, HEXABITZ_USER_INTERFACE_PARTS:VLMS1300-GS08
- added D12, D13: Green, HEXABITZ_USER_INTERFACE_PARTS:VLMTG1300-GS08
- added R10, R11, R31, R9: 270.0R, HEXABITZ_RCLS:R-0603
- added R33, R34: DNP, HEXABITZ_RCLS:R-0603
- added U3: TEXAS_INSTRUMENTS_ISO7741DBQRTEXAS_INSTRUMENTS_ISO7741DBQR_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, HEXABITZ_ICs:TEXAS_INSTRUMENTS_ISO7741DBQRTEXAS_INSTRUMENTS_ISO7741DBQR_0_0
- C5: device HEXABITZ_RCLS:C-0805 -> HEXABITZ_RCLS:C-0603
- D0: value VLMS1300-GS08 -> RED; device Hexabitz:VLMS1300-GS08 -> HEXABITZ_USER_INTERFACE_PARTS:VLMS1300-GS08
- D2: value red -> RED; device HEXABITZ_USER_INTERFACE_PARTS:LEDCHIP-LED0805 -> HEXABITZ_USER_INTERFACE_PARTS:VLMS1300-GS08; DESCRIPTION LED Uni-Color Red Orange 630nm 2-Pin SMD T/R -> (none)
- D3, D4, D5, D6, D7: value yallow -> YELLOW; device HEXABITZ_USER_INTERFACE_PARTS:LEDCHIP-LED0805 -> HEXABITZ_USER_INTERFACE_PARTS:VLMY1300-GS08; DESCRIPTION Yellow 2 x 1.25 x 1.1 mm 130° Water Clear 2.5 mcd 2.1 V LED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 -> (none)
- D8: value green -> Green; device HEXABITZ_USER_INTERFACE_PARTS:LEDCHIP-LED0805 -> HEXABITZ_USER_INTERFACE_PARTS:VLMTG1300-GS08; DESCRIPTION Green 2 x 1.25 x 1.1 mm 130° Water Clear 6 mcd 2.1 V SMT LED -> (none)
- P1: value HEXABIT__X3_NO_P1_P2_P3_P4 -> HEXABIT__X3_NO_P1_P2_P3_P4_P5_P6_P11_P12; device hexabitz_connectors:HEXABIT__X3_NO_P1_P2_P3_P4 -> hexabitz_connectors:HEXABIT__X3_NO_P1_P2_P3_P4_P5_P6_P11_P12
- R22, R27: device HEXABITZ_RCLS:R-0805 -> HEXABITZ_RCLS:R-0603
- renumbered J1 to EMG_SW, R50 to R32
Connections:
- removed net SPI2_CS: U1.PB12
- removed net UART5_RX: P1.SD11
- removed net UART5_TX: P1.SU11
- removed net VDDIO: U2A.VDDIO
- new net FORWARD: R10.2, U1.PB12
- new net N$24: D12.A, R10.1
- new net N$25: D13.A, R11.1
- new net REVERSED: R11.2, U1.PA12
- new net STOPPED: R9.2, U1.PA11
- net BUSY/SYNC: now also U6.OUTA; no longer U6.INC
- net CK: now also U3.OUTB; no longer U5.OUTB
- net CS: now also U3.OUTA; no longer U5.OUTA
- net FLAG: now also U6.OUTB; no longer U6.IND
- net GND: now also C21.2, C22.-, C23.-, C24.-, C25.2, C26.2, C27.2, C28.2, C29.2, D11.C, D12.C, D13.C, U1.PC12, U1.PD2, U3.1_GND1, U3.2_GND1; no longer C100.2, C200.-, C300.2, C400.-, C50.2, C500.2, C600.2, C700.-, C900.2, P1.GND1, P1.GND10, P1.GND11, P1.GND12, P1.GND5, P1.GND6, U1.PA11, U1.PA12, U5.1_GND1, U5.2_GND1
- net GND1: now also U3.1_GND2, U3.2_GND2; no longer U5.1_GND2, U5.2_GND2
- net MC_BUSY/SYNC: now also U1.PC5; no longer U1.PA6
- net MC_CK: now also U3.INB; no longer U5.INB
- net MC_CS: now also U3.INA; no longer U5.INA
- net MC_FLAG: now also U1.PC4; no longer U1.PA7
- net MC_MISO: now also R33.1, U3.OUTD; no longer U5.OUTD
- net MC_MOSI: now also R34.1, U3.INC; no longer U5.INC
- net MC_STBY/RESET: now also U1.PA6; no longer U1.PC5
- net MS_STCK: now also U1.PA7; no longer U1.PC4
- net N$11: now also D11.A, R9.1; no longer R16.2, R17.2, R18.2, R19.2
- net N$18: now also U3.OUTC; no longer U5.OUTC
- net N$19: now also U3.IND; no longer U5.IND
- net N$3: now also R31.2; no longer R100.2
- net N$4: now also R31.1; no longer R100.1
- net OUTA1: now also R16.2, X3-2.KL; no longer X3-1.KL
- net OUTA2: now also R17.2, X3-1.KL; no longer X3-2.KL
- net OUTB1: now also R18.2
- net OUTB2: now also R19.2
- net R1: now also C21.1; no longer C50.1
- net STBY/RESET: now also U6.IND; no longer U6.OUTB
- net STCK: now also U6.INC; no longer U6.OUTA
- net UART1_RX*: now also P1.SD9; no longer P1.SD10
- net UART1_TX*: now also P1.SU9; no longer P1.SU10
- net UART3_RX: no longer P1.SD9
- net UART3_TX: no longer P1.SU9
- net UART4_RX: now also P1.SD10, U1.PC11; no longer P1.SD6, U1.PA1
- net UART4_TX: now also P1.SU10, U1.PC10; no longer P1.SU6, U1.PA0
- net UART7_RX: no longer P1.SD12
- net UART7_TX: no longer P1.SU12
- net UART8_RX: no longer P1.SD5
- net UART8_TX: no longer P1.SU5
- net VCCIO: now also C1.1, C16.1, C18.1, C4.1, R13.2, R14.2, R15.1, R21.2, R25.2, R26.2, U2A.VDDIO, U3.EN2, U3.VCC2; no longer U5.EN2, U5.VCC2
- net VDD: now also C22.+, C23.+, C24.+, C25.1, C26.1, C27.1, C28.1, C29.1, R33.2, R34.2, U3.EN1, U3.VCC1; no longer C1.1, C100.1, C16.1, C18.1, C200.+, C300.1, C4.1, C400.+, C500.1, C600.1, C700.+, C900.1, P1.VDD1, P1.VDD10, P1.VDD11, P1.VDD12, P1.VDD5, P1.VDD6, R13.2, R14.2, R15.1, R21.2, R25.2, R26.2, U5.EN1, U5.VCC1

Commit message: no message
Parts:
- added P3, P4, P5, P6, VCCIO, VCCIO1, VS: PAD4, HEXABITZ_CONNECTION_PARTS:PAD4
- renumbered D11 to S, D12 to CCW, D13 to CW, D2 to FLT, D3 to A1, D4 to A2, D5 to B1, D6 to B2, D7 to BZY, D8 to PWR, U6 to U4
Connections:
- removed net SPI2_MISO: U1.PB14
- removed net SPI2_SCK: U1.PB13
- net GND: now also P5.P$1
- net GND1: now also P6.P$1
- net VCCIO: now also VCCIO.P$1, VCCIO1.P$1
- net VDD: now also P4.P$1
- net VSS: now also VS.P$1
Other:
- note added: "isolated Stepper motor driver 10A , 10.5 to 80V"
- note removed: "Stepper motor driver 10A , 10.5 to 50V"
- moved on the sheet: C5, EMG_SW, R1, R2, R27, R28, X2-1, X2-2, X3-1, X3-2, X4-1, X4-2
