File: H17R10/design/H17R10.brd (EAGLE design)
At the start: 60 x 60.6 mm, 72 parts, among them J1 3-644456-2, U1 STM32G0B1CEU6NUFQFPN48_STM32_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, U2 POWERSTEP01, X1 8MHZ

Commit message: -Replace the blind vias with through hole ones
Routing:
- net BUSY/SYNC: track 24.4 -> 29.3 mm
- net OUTB1: track 24.7 -> 26.5 mm
- net VSSA: track 115.3 -> 116.8 mm
- net OUTA1: track 23.1 -> 22.2 mm
- net SENSEB: vias 15 -> 7
- net SENSEA: vias 15 -> 7
- removed copper zone on layer 2, net SENSEA
- removed copper zone on layer 2, net SENSEB
