File: H17R10/design/H17R10.sch (EAGLE design)
At the start: 72 parts, among them J1 3-644456-2, P1 HEXABIT_17.32_X3_NO_P1_P2_P3_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, U1 STM32G0B1CEU6NUFQFPN48_STM32_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, U2 POWERSTEP01, X1 8MHZ

Commit message: -Connect missing wires - Delete power led - Improve the layout for better performance and appearance
Parts:
- removed D9: Green, HEXABITZ_USER_INTERFACE_PARTS:VLMTG1300-GS08
- removed JP2: (no value), pinhead:PINHD-1X3
- removed R12: 330, HEXABITZ_RCLS:R-0603
- added SWD: (no value), pinhead:PINHD-1X3
- C21: device HEXABITZ_RCLS:C-0805-POL -> HEXABITZ_RCLS:T491A226K006AT; MFN KEMET -> (none); MPN T491A226K006AT -> (none); OCTOPART_URL https://octopart.com/t491a226k006at-kemet-968601?r=sp -> (none); VOLTAGE_RATING 6.3V -> (none)
- renumbered J1 to EMG_SW, JP1 to R, P1 to U$1, SJ1 to SA_J, SJ2 to SB_J, X2 to PWR, X3 to A, X4 to B
Connections:
- removed net N$14: D9.A, R12.1
- net BUSY/SYNC: now also U1.PA12[PA10]
- net C: now also SWD.1, SWD.2; no longer JP2.1, JP2.2
- net D: now also SWD.3; no longer JP2.3
- net FLAG: now also U1.PA11[PA9]
- net GND: now also U$1.GND1, U$1.GND2, U$1.GND3; no longer U$1.GND7, U$1.GND8, U$1.GND9
- net RESET: now also U1.PB6
- net STCK: now also U1.PB7
- net USART2_RX: now also U$1.SD2; no longer U$1.SD8
- net USART2_TX: now also U$1.SU2; no longer U$1.SU8
- net USART3_RX: now also U$1.SD3; no longer U$1.SD9
- net USART3_TX: now also U$1.SU3; no longer U$1.SU9
- net USART5_RX: now also U$1.SD4; no longer U$1.SD10
- net USART5_TX: now also U$1.SU4; no longer U$1.SU10
- net USART6_RX: now also U$1.SD1; no longer U$1.SD7
- net USART6_TX: now also U$1.SU1; no longer U$1.SU7
- net VDD: now also U$1.VDD1, U$1.VDD2, U$1.VDD3; no longer U$1.VDD7, U$1.VDD8, U$1.VDD9
- net VDDA: no longer R12.2
- net VSSA: no longer D9.C
Other:
- note removed: "R"
- note removed: "VDD = 3.3 Volts"
- moved on the sheet: R3
